File: EC1834_FDC.kicad_sch (KiCad schematic)
At the start: 125 parts, among them K1 100n, K3 100n, K32 100n, Q1 8000kHz, SW1 SW_DIP_x02, SW2 SW_DIP_x08, X1 BUS_EC1834_16Bit, X2 X2, X3 X3, X4 X4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

Commit message: Bugfix in schematics documented
Other:
- note added: "X"
- note added: "X = Fehler im rekonstruierten Originalschaltplan!"
Changed lines of the file:
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@@
+		)
+	)
+	(text "X"
+		(exclude_from_sim no)
+		(at 277.114 149.606 0)
+		(effects
+			(font
+				(size 2.5 2.5)
+				(thickness 0.8)
+				(bold yes)
+				(color 255 0 0 1)
+			)
+		)
+	)
+	(text "X = Fehler im rekonstruierten \nOriginalschaltplan!"
+		(exclude_from_sim no)
+		(at 141.224 323.85 0)
+		(effects
+			(font
+				(size 2 2)
+				(thickness 0.4)
+				(bold yes)
+				(color 194 0 0 1)
+			)
 		)
 	)

Commit message: Schematics improved Added descriptions Fixed last missing PCB components
Parts:
- removed SW1: SW_DIP_x02, Button_Switch_THT:SW_DIP_SPSTx02_Slide_9.78x7.26mm_W7.62mm_P2.54mm, symbol Switch:SW_DIP_x02
- added S2_1: DEF_OFF, Button_Switch_THT:SW_DIP_SPSTx01_Slide_9.78x4.72mm_W7.62mm_P2.54mm, symbol Switch:SW_DIP_x01
- added S2_2: DEF_ON, Button_Switch_THT:SW_DIP_SPSTx01_Slide_9.78x4.72mm_W7.62mm_P2.54mm, symbol Switch:SW_DIP_x01
- C12, C13, C16, C17, C19, C20: now not fitted; now left out of the parts list
- renumbered SW2 to S1
Connections:
- net at A12.14 (~{Q4}), A3.1 (CS), A40.9 (A3): now also S2_1.2
- net at A17.2 (B1), A17.4 (A2), A40.8 (Y3)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: now also S2_2.2
- net at A10.3 (B1): now also S2_1.1, S2_2.1
Other:
- note added: "Conf Reg 3F4"
- note added: "Ctrl Reg 3F4"
- note added: "Data Read"
- note added: "Data Write"
- note added: "IO Port 0x3F4"
- note added: "IO Port 0x3F_"
- note added: "IO WR 0x3F4"
- note added: "PLL"
- note added: "PreComp"
- note added: "Takterzeugung TA8 8Mhz TA4 4MHz TA3 2,666MHz TA2 2MHz"
- note added: "X5 Messpunkte X5:1 - PLL 2000kHz ±2kHz X5:2 - Data Window (mit X5:4) X5:3 - ? X5:4 - Read Data (mit X5:2) X5:5 - n/v"
- moved on the sheet: A15B, A16A, A16B, A17C, A27F, A30D, A33B, A38D, A40D, C3, C4, C5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
