File: Power.kicad_sch (KiCad schematic)
At the start: 87 parts, among them K10 100n, K11 100n, K12 100n, K13 100n, K14 100n, K15 100n, K16 100n, K17 100n, K18 100n, K19 100n, K2 100n, K20 100n, K21 100n, K22 100n, K23 100n, K24 100n, K25 100n, K26 100n, K27 100n, K28 100n, K29 100n, K30 100n, K31 100n, K33 100n, K34 100n, K35 100n, K36 100n, K37 100n, K38 100n, K39 100n, K4 100n, K40 100n, K41 100n, K42 100n, K43 100n, K44 100n, K5 100n, K6 100n, K7 100n, K8 100n, K9 100n

Commit message: Schematics improved Added descriptions Fixed last missing PCB components
Parts:
- added W1, W2: W1, TestPoint:TestPoint_Bridge_Pitch2.54mm_Drill0.7mm, symbol Connector:TestPoint_2Pole
Connections:
- net GND: now also W1.1, W1.2, W2.1, W2.2
Changed lines of the file:
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@@
 	)
 	(junction
+		(at 311.15 59.69)
+		(diameter 0)
+		(color 0 0 0 0)
+	)
+	(junction
 		(at 234.95 93.98)
 		(diameter 0)
@@
 	)
 	(junction
+		(at 321.31 50.8)
+		(diameter 0)
+		(color 0 0 0 0)
+	)
+	(junction
 		(at 102.87 111.76)
 		(diameter 0)
@@
 	)
 	(junction
+		(at 321.31 59.69)
+		(diameter 0)
+		(color 0 0 0 0)
+	)
+	(junction
 		(at 260.35 111.76)
 		(diameter 0)
@@
 	)
 	(junction
+		(at 311.15 50.8)
+		(diameter 0)
+		(color 0 0 0 0)
+	)
+	(junction
 		(at 191.77 77.47)
 		(diameter 0)
@@
 	(wire
 		(pts
+			(xy 321.31 50.8) (xy 325.12 50.8)
+		)
+		(stroke
+			(width 0)
+			(type default)
+		)
+	)
+	(wire
+		(pts
+			(xy 321.31 50.8) (xy 321.31 59.69)
+		)
+		(stroke
+			(width 0)
+			(type default)
+		)
+	)
+	(wire
+		(pts
 			(xy 204.47 43.18) (xy 210.82 43.18)
 		)
@@
 	(wire
 		(pts
+			(xy 311.15 50.8) (xy 311.15 59.69)
+		)
+		(stroke
+			(width 0)
+			(type default)
+		)
+	)
+	(wire
+		(pts
 			(xy 87.63 91.44) (xy 87.63 93.98)
 		)
@@
 	(wire
 		(pts
+			(xy 311.15 59.69) (xy 311.15 67.31)
+		)
+		(stroke
+			(width 0)
+			(type default)
+		)
+	)
+	(wire
+		(pts
 			(xy 226.06 91.44) (xy 226.06 93.98)
 		)
@@
 	(wire
 		(pts
+			(xy 321.31 59.69) (xy 321.31 67.31)
+		)
+		(stroke
+			(width 0)
+			(type default)
+		)
+	)
+	(wire
+		(pts
 			(xy 59.69 43.18) (xy 67.31 43.18)
 		)
@@
 	(wire
 		(pts
-			(xy 309.88 50.8) (xy 317.5 50.8)
+			(xy 309.88 50.8) (xy 311.15 50.8)
 		)
 		(stroke
@@
 	(wire
 		(pts
-			(xy 317.5 50.8) (xy 325.12 50.8)
+			(xy 317.5 50.8) (xy 321.31 50.8)
 		)
 		(stroke
@@
 	(wire
 		(pts
+			(xy 311.15 50.8) (xy 317.5 50.8)
+		)
+		(stroke
+			(width 0)
+			(type default)
+		)
+	)
+	(wire
+		(pts
 			(xy 63.5 77.47) (xy 76.2 77.47)
 		)
@@
 	)
 	(symbol
+		(lib_id "Connector:TestPoint_2Pole")
+		(at 316.23 59.69 0)
+		(unit 1)
+		(exclude_from_sim no)
+		(in_bom yes)
+		(on_board yes)
+		(dnp no)
+		(fields_autoplaced yes)
+		(property "Reference" "W1"
+			(at 316.23 54.9105 0)
+			(effects
+				(font
+					(size 1.27 1.27)
+				)
+			)
+		)
+		(property "Value" "W1"
+			(at 316.23 57.3348 0)
+			(effects
+				(font
+					(size 1.27 1.27)
+				)
+			)
+		)
+		(property "Footprint" "TestPoint:TestPoint_Bridge_Pitch2.54mm_Drill0.7mm"
+			(at 316.23 59.69 0)
+			(effects
+				(font
+					(size 1.27 1.27)
+				)
+				(hide yes)
+			)
+		)
+		(property "Datasheet" "~"
+			(at 316.23 59.69 0)
+			(effects
+				(font
+					(size 1.27 1.27)
+				)
+				(hide yes)
+			)
+		)
+		(property "Description" "2-polar test point"
+			(at 316.23 59.69 0)
+			(effects
+				(font
+					(size 1.27 1.27)
+				)
+				(hide yes)
+			)
+		)
+		(pin "1"
+		)
+		(pin "2"
+		)
+		(instances
+			(project ""
+				(path "/bbd6417a-5f3d-4c8e-910d-4ce325bd4790/00000000-0000-0000-0000-000063239fae"
+					(reference "W1")
+					(unit 1)
+				)
+			)
+		)
+	)
+	(symbol
 		(lib_id "robotron_ec1834:DL074")
 		(at 82.55 124.46 0)
@@
 					(unit 1)
 				)
+			)
+		)
+	)
+	(symbol
+		(lib_id "Connector:TestPoint_2Pole")
+		(at 316.23 67.31 0)
+		(unit 1)
+		(exclude_from_sim no)
+		(in_bom yes)
+		(on_board yes)
+		(dnp no)
+		(fields_autoplaced yes)
+		(property "Reference" "W2"
+			(at 316.23 62.5305 0)
+			(effects
+				(font
+					(size 1.27 1.27)
+				)
+			)
+		)
+		(property "Value" "W1"
+			(at 316.23 64.9548 0)
+			(effects
+				(font
+					(size 1.27 1.27)
+				)
+			)
+		)
+		(property "Footprint" "TestPoint:TestPoint_Bridge_Pitch2.54mm_Drill0.7mm"
+			(at 316.23 67.31 0)
+			(effects
+				(font
+					(size 1.27 1.27)
+				)
+				(hide yes)
+			)
+		)
+		(property "Datasheet" "~"
+			(at 316.23 67.31 0)
+			(effects
+				(font
+					(size 1.27 1.27)
+				)
+				(hide yes)
+			)
+		)
+		(property "Description" "2-polar test point"
+			(at 316.23 67.31 0)
+			(effects
+				(font
+					(size 1.27 1.27)
+				)
+				(hide yes)
+			)
+		)
+		(pin "1"
+		)
+		(pin "2"
+		)
+		(instances
+			(project "EC1834-FDC"
+				(path "/bbd6417a-5f3d-4c8e-910d-4ce325bd4790/00000000-0000-0000-0000-000063239fae"
+					(reference "W2")
+					(unit 1)
+				)
